File: OpAmpTester.kicad_sch (KiCad schematic)
At the start: 56 parts, among them J1 V-IN, U1 DUT, U2 DUT, U3 DUT

Commit message: BOM file
Parts:
- C1: value 10U -> (none); footprint -lmp-misc:CP_Radial_D5.0mm_P2.50mm -> (none); Distributor (none) -> Mouser; DistributorPartLink (none) -> https://www.mouser.ca/ProductDetail/Panasonic/ECA-1EM100I?q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; DistributorPartNum (none) -> 667-ECA-1EM100I; Manufacturer (none) -> Panasonic; ManufacturerPartNum (none) -> ECA-1EM100I
- C10, C11, C12, C2, C5, C6, C9: value 1U -> (none); footprint -lmp-misc:CP_Radial_D4.0mm_P2.50mm -> (none); Distributor (none) -> Mouser; DistributorPartLink (none) -> https://www.mouser.ca/ProductDetail/Lelon/SEA010M1HBK-0407P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; DistributorPartNum (none) -> 140-SEA1R0M1HBK0407; Manufacturer (none) -> Lelon; ManufacturerPartNum (none) -> SEA010M1HBK-0407P
- C13, C14, C3, C4, C7, C8: value 100N -> (none); footprint -lmp-misc:C_Disc_D5.0mm_W2.5mm_P2.50mm -> (none); Note IC decoupling -> (none)
- D1: value 1N4001 -> (none); footprint Diode_THT:D_DO-41_SOD81_P10.16mm_Horizontal -> (none); Distributor (none) -> Mouser; DistributorPartLink (none) -> https://www.mouser.ca/ProductDetail/onsemi/1N4001RLG?qs=y2k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; DistributorPartNum (none) -> 863-1N4001RLG; Manufacturer (none) -> onsemi; ManufacturerPartNum (none) -> 1N4001RLG
- D2, D3, D4, D5, D6, D7, D8: value LED -> (none); footprint LED_THT:LED_D3.0mm -> (none); Distributor (none) -> Mouser; DistributorPartLink (none) -> https://www.mouser.ca/ProductDetail/Lite-On/LTL-1CHE?qs=sGA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; DistributorPartNum (none) -> 859-LTL-1CHE; Manufacturer (none) -> Lite-On; ManufacturerPartNum (none) -> LTL-1CHE
- J1: value V-IN -> (none); footprint Connector_PinSocket_2.54mm:PinSocket_1x02_P2.54mm_Vertical -> (none); Distributor (none) -> Adafruit; Distributor2 (none) -> Mouser; DistributorPartLink (none) -> https://www.adafruit.com/product/598; DistributorPartLink2 (none) -> https://www.mouser.ca/ProductDetail/Wurth-Elektronik/613032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; DistributorPartNum (none) -> 598; DistributorPartNum2 (none) -> 710-61303211821
- R1, R10, R14, R18, R2, R22, R26, R30, R6: value 1K -> (none); footprint -lmp-misc:R_Axial_DIN0207_L6.3mm_D2.5mm_P10.16mm_Horizontal -> (none); DistributorPartLink https://www.mouser.ca/c/passive-components/resistors/film-r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 -> https://www.mouser.ca/ProductDetail/Vishay-Dale/CCF071K00JK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; DistributorPartNum 603-MFR-12* -> 71-CCF071K00JKE36; Manufacturer YAGEO -> Vishay / Dale; ManufacturerPartNum MFR-12* -> CCF071K00JKE36; Value2 1%, 1/6 W -> (none)
- R11, R12, R13, R15, R16, R17, R19, R20, R21, R23, R24, R25, R27, R28, R29, R3, R4, R5, R7, R8, R9: value 100K -> (none); footprint -lmp-misc:R_Axial_DIN0207_L6.3mm_D2.5mm_P7.62mm_Horizontal -> (none); DistributorPartLink https://www.mouser.ca/c/passive-components/resistors/film-r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 -> https://www.mouser.ca/ProductDetail/YAGEO/MFR-12FTF52-100K?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; DistributorPartNum 603-MFR-12* -> 603-MFR-12FTF52-100K; ManufacturerPartNum MFR-12* -> MFR-12FTF52-100K; Value2 1%, 1/6 W -> (none)
- U1: value DUT -> (none); footprint Package_DIP:DIP-8_W7.62mm_Socket -> (none); Distributor Digi-Key -> Mouser; Distributor2 Mouser -> (none); DistributorPartLink https://www.digikey.ca/en/products/detail/texas-instruments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 -> https://www.mouser.ca/ProductDetail/Mill-Max/110-47-308-41-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; DistributorPartLink2 https://www.mouser.ca/ProductDetail/Texas-Instruments/TL071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 -> (none); DistributorPartNum 296-34258-5-ND -> 575-1104730841001000; DistributorPartNum2 595-TL071IPE4 -> (none); Manufacturer Texas Instruments -> Mill-Max; ManufacturerPartNum TL071BCP -> 110-47-308-41-001000; Note (none) -> Socket only
- U2: value DUT -> (none); footprint Package_DIP:DIP-8_W7.62mm_Socket -> (none); DistributorPartLink https://www.mouser.ca/ProductDetail/Texas-Instruments/TL072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 -> https://www.mouser.ca/ProductDetail/Mill-Max/110-47-308-41-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; DistributorPartNum 595-TL072BCP -> 575-1104730841001000; Manufacturer Texas Instruments -> Mill-Max; ManufacturerPartNum TL072BCP -> 110-47-308-41-001000; Note (none) -> Socket only
- U3: value DUT -> (none); footprint Package_DIP:DIP-14_W7.62mm_Socket -> (none); DistributorPartLink https://www.mouser.ca/ProductDetail/?qs=vxEfx8VrU7BHurOY5iQ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 -> https://www.mouser.ca/ProductDetail/Mill-Max/110-47-314-41-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; DistributorPartNum 595-TL074BCN -> 575-1104731441001000; Manufacturer Texas Instruments -> Mill-Max; ManufacturerPartNum TL074BCN -> 110-47-314-41-001000; Note (none) -> Socket only
