File: OpAmpTester.kicad_sch (KiCad schematic)
At the start: 56 parts

Commit message: schematic tweaks
Parts:
- C1: value (none) -> 10U; footprint (none) -> -lmp-misc:CP_Radial_D5.0mm_P2.50mm
- C10, C11, C12, C2, C5, C6, C9: value (none) -> 1U; footprint (none) -> -lmp-misc:CP_Radial_D4.0mm_P2.50mm
- C13, C14, C3, C4, C7, C8: value (none) -> 100N; footprint (none) -> -lmp-misc:C_Disc_D5.0mm_W2.5mm_P2.50mm
- D1: value (none) -> 1N4001; footprint (none) -> Diode_THT:D_DO-41_SOD81_P10.16mm_Horizontal
- D2, D3, D4, D5, D6, D7, D8: value (none) -> LED; footprint (none) -> LED_THT:LED_D3.0mm
- J1: value (none) -> V-IN; footprint (none) -> Connector_PinSocket_2.54mm:PinSocket_1x02_P2.54mm_Vertical
- R1, R10, R14, R18, R2, R22, R26, R30, R6: value (none) -> 1K; footprint (none) -> -lmp-misc:R_Axial_DIN0207_L6.3mm_D2.5mm_P10.16mm_Horizontal
- R11, R12, R13, R15, R16, R17, R19, R20, R21, R23, R24, R25, R27, R28, R29, R3, R4, R5, R7, R8, R9: value (none) -> 100K; footprint (none) -> -lmp-misc:R_Axial_DIN0207_L6.3mm_D2.5mm_P7.62mm_Horizontal
- U1, U2: value (none) -> DUT; footprint (none) -> Package_DIP:DIP-8_W7.62mm_Socket
- U3: value (none) -> DUT; footprint (none) -> Package_DIP:DIP-14_W7.62mm_Socket
Other:
- moved on the sheet: C10, C11, C12, C5, C6, C9
