File: OpAmpTester.kicad_pcb (KiCad board)
At the start: 2 copper layers, 48.9 x 80 mm, 58 parts, among them J1 V-IN, U1 DUT, U2 DUT, U3 DUT

Commit message: Add pin-1 indicators for sockets
Other:
- board text added: "rev ${REVISION}"
- board text removed: "rev 1.0"
Changed lines of the file:
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@@
   (title_block
     (title "Op Amp Tester")
-    (date "2022-04-20")
-    (rev "1.0")
+    (date "2022-07-06")
+    (rev "1.01")
     (company "Len Popp")
     (comment 1 "Copyright © 2022 Len Popp CC BY")
@@
     )
   )
+  (gr_circle (center 128.865 69.85) (end 129.5 69.85) (layer "F.SilkS") (width 0.12) (fill solid))
+  (gr_circle (center 128.865 109.22) (end 129.5 109.22) (layer "F.SilkS") (width 0.12) (fill solid))
+  (gr_circle (center 128.865 87.63) (end 129.5 87.63) (layer "F.SilkS") (width 0.12) (fill solid))
   (gr_rect (start 114.3 55.88) (end 163.195 135.89) (layer "Edge.Cuts") (width 0.05) (fill none))
   (gr_text "B" (at 156.21 132.08) (layer "F.SilkS")
     (effects (font (size 1.27 1.27) (thickness 0.254)) (justify left))
   )
-  (gr_text "rev 1.0" (at 147.955 60.325) (layer "F.SilkS")
+  (gr_text "rev ${REVISION}" (at 147.955 60.325) (layer "F.SilkS")
     (effects (font (size 1 1) (thickness 0.15)) (justify left))
   )
